File: PantryLED.kicad_sch (KiCad schematic)
At the start: 20 parts, among them J1 Conn_01x06_Male, U1 LM2576HVS-3.3, U2 VN2106N3-G, U3 MSP430G2202IN20

Commit message: put back R2
Parts:
- R2: value 1k -> 47k
Connections:
- no-connect marks 0 -> 2
Other:
- note added: "2024/09/02: Replaced buck converter with same family but with 3.3V output short R3 and remove R4"
- note added: "RST pullup"
Changed lines of the file:
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@@
   (junction (at 77.47 71.12) (diameter 0) (color 0 0 0 0)
   )
+  (no_connect (at 109.22 67.31))
+  (no_connect (at 109.22 55.88))
   (wire (pts (xy 166.37 107.95) (xy 189.23 107.95))
     (stroke (width 0) (type default) (color 0 0 0 0))
@@
   (wire (pts (xy 38.1 59.69) (xy 38.1 71.12))
     (stroke (width 0) (type default) (color 0 0 0 0))
+  )
+  (text "RST pullup " (at 102.87 88.9 0)
+    (effects (font (size 1.27 1.27)) (justify left bottom))
+  )
+  (text "2024/09/02: Replaced buck converter with same family but with 3.3V output\nshort R3 and remove R4"
+    (at 36.83 26.67 0)
+    (effects (font (size 1.27 1.27)) (justify left bottom))
   )
   (text "12V Rail\nGND_12\nLiDAR Input\nSBWTCK\nSBWTDIO\n3.3V Rail\nGND\n"
@@
       (effects (font (size 1.27 1.27)) (justify left))
     )
-    (property "Value" "1k" (id 1) (at 111.76 93.9799 0)
+    (property "Value" "47k" (id 1) (at 111.76 93.9799 0)
       (effects (font (size 1.27 1.27)) (justify left))
     )
@@
     )
     (path "/1f4347b8-2b82-4f0b-b355-55697015b9aa"
-      (reference "R2") (unit 1) (value "1k") (footprint "Resistor_THT:R_Axial_DIN0207_L6.3mm_D2.5mm_P10.16mm_Horizontal")
+      (reference "R2") (unit 1) (value "47k") (footprint "Resistor_THT:R_Axial_DIN0207_L6.3mm_D2.5mm_P10.16mm_Horizontal")
     )
     (path "/f48e6cca-db2b-49b1-a586-40b405680efb"
